Commit message: ray detection is 10000times faster

File: rsc/megabot/smb.urdf (robot description, URDF)
Before this commit: robot smb, 7 links, 6 joints
Links:
- added link lidar; visual cylinder length=0.2 radius=0.05
Joints:
- added joint lidar: type fixed, parent base, child lidar, origin xyz=0 0 0.2 rpy=0 0 0
