Commit message: mjcf wip. examples added

File: rsc/kinova/urdf/kinova.urdf (robot description, URDF)
Before this commit: robot kinova, 16 links, 15 joints
Links:
- removed link kinova_link_finger_1
- removed link kinova_link_finger_2
- removed link kinova_link_finger_3
- removed link kinova_link_finger_tip_1
- removed link kinova_link_finger_tip_2
- removed link kinova_link_finger_tip_3
- link kinova_end_effector: geometry visual box size=0.0001 0.0001 0.0001
- link kinova_link_1: geometry visual mesh filename=../meshes/ring_big.STL; visual mesh filename=../meshes/shoulder.dae
- link kinova_link_2: geometry visual mesh filename=../meshes/arm.dae; visual mesh filename=../meshes/ring_big.STL
- link kinova_link_3: geometry visual mesh filename=../meshes/forearm.dae; visual mesh filename=../meshes/ring_big.STL
- link kinova_link_4: geometry visual mesh filename=../meshes/ring_small.STL; visual mesh filename=../meshes/wrist_spherical_1.dae
- link kinova_link_5: geometry visual mesh filename=../meshes/ring_small.STL; visual mesh filename=../meshes/wrist_spherical_2.dae
- link kinova_link_6: geometry visual mesh filename=../meshes/hand_3finger.dae; visual mesh filename=../meshes/ring_small.STL
- link kinova_link_base: geometry visual mesh filename=../meshes/base.dae
Joints:
- removed joint kinova_joint_finger_1
- removed joint kinova_joint_finger_2
- removed joint kinova_joint_finger_3
- removed joint kinova_joint_finger_tip_1
- removed joint kinova_joint_finger_tip_2
- removed joint kinova_joint_finger_tip_3
