Commit message: 1. add debug_app.cpp with my modified 2. ppo.py with clip output 3. raisim_gym_helper.py got a Logger using logging which could save your log in both .log and console 4. design my self Environment.hpp and could read configuration to simplify your training with less compilation

File: rsc/anymal_c/urdf/anymal.urdf (robot description, URDF)
Before this commit: robot anymal, 78 links, 77 joints
Joints:
- joint LF_HFE: limit lower=-9.42477796077 upper=9.42477796077 effort=80.0 velocity=7.5 -> lower=-0.5 upper=2 effort=80.0 velocity=7.5
- joint LF_KFE: limit lower=-9.42477796077 upper=9.42477796077 effort=80.0 velocity=7.5 -> lower=-3.15 upper=0.5 effort=80.0 velocity=7.5
- joint LH_HFE: limit lower=-9.42477796077 upper=9.42477796077 effort=80.0 velocity=7.5 -> lower=-2 upper=0.5 effort=80.0 velocity=7.5
- joint LH_KFE: limit lower=-9.42477796077 upper=9.42477796077 effort=80.0 velocity=7.5 -> lower=-0.5 upper=3.15 effort=80.0 velocity=7.5
- joint RF_HFE: limit lower=-9.42477796077 upper=9.42477796077 effort=80.0 velocity=7.5 -> lower=-0.5 upper=2 effort=80.0 velocity=7.5
- joint RF_KFE: limit lower=-9.42477796077 upper=9.42477796077 effort=80.0 velocity=7.5 -> lower=-3.15 upper=0.5 effort=80.0 velocity=7.5
- joint RH_HFE: limit lower=-9.42477796077 upper=9.42477796077 effort=80.0 velocity=7.5 -> lower=-2 upper=0.5 effort=80.0 velocity=7.5
- joint RH_KFE: limit lower=-9.42477796077 upper=9.42477796077 effort=80.0 velocity=7.5 -> lower=-0.5 upper=3.15 effort=80.0 velocity=7.5
