Commit message: changed the lidar output to 3d points

File: raisim/win32/bin/rsc/anymal_c/urdf/anymal_sensored.urdf (robot description, URDF)
Before this commit: robot anymal, 78 links, 77 joints
Links:
- added link lidar_link
Joints:
- added joint base_to_lidar: type fixed, parent base, child lidar_link, origin xyz=0.0 0.0 0.08 rpy=0.0 0.0 0.0
